File: fanpower.kicad_pcb (KiCad board)
At the start: 2 copper layers, 22 parts, among them J1 Conn_01x06, J2 Conn_01x03, J3 Conn_01x02, J4 Conn_01x04, J5 Conn_01x04, Q1 BSH105,215, Q2 BSH105,215, SW1 SW_SPDT, SW2 SW_SPDT, U1 R-78E5.0-0.5

Commit message: Add FLOW measurement.
Parts:
- removed J1: Conn_01x06, Connector_PinHeader_2.54mm:PinHeader_1x06_P2.54mm_Vertical
- removed R3: 2k, Resistor_SMD:R_0805_2012Metric
- added FLOW1: Conn_01x02, Connector_PinHeader_2.54mm:PinHeader_1x02_P2.54mm_Vertical, F.Cu at (193.7, 87.0)
- R2: value 2k -> 10k
- moved R9 13.2 mm to (206.8, 103.1)
- moved SW2 12.1 mm to (193.7, 104.4)
- moved R7 7.62 mm to (203.7, 103.1), turned to 90 degrees
- moved FAN2 5.72 mm to (198.8, 108.0)
- moved NTC1 4.71 mm to (204.2, 87.0)
- moved R8 3.56 mm to (201.7, 103.1), turned to 90 degrees
- moved Q2 2.54 mm to (198.6, 103.1), turned to 180 degrees
- moved R2 2.36 mm to (197.5, 87.0)
- moved R1 2.07 mm to (208.3, 87.0)
- renumbered J4 to FAN1, J5 to FAN2, J3 to NTC1
Connections:
- A1 pad 14: /SIGON2 -> Net-(A1-Pad14)
- A1 pad 17: /I2C_SCL -> /SIGTACH1
- A1 pad 18: /I2C_SDA -> /SIGON1
- A1 pad 5: /SIGON1 -> /SIGON2
- A1 pad 6: /SIGTACH1 -> /SIGTACH2
- A1 pad 7: /SIGTACH2 -> /FLOW
- R2 pad 2: /I2C_SCL -> /FLOW
Routing:
- net +3V3: track 0.00 -> 63.6 mm, vias 0 -> 4
- net /FLOW: track 0.00 -> 40.1 mm
- net /SIGTACH2: track 26.0 -> 8.28 mm
- net /SIGON1: track 26.4 -> 12.1 mm
- net /NTC: track 0.00 -> 11.9 mm
- net /SIGTACH1: track 27.3 -> 20.2 mm
- net /SIGPWM2: track 21.1 -> 26.0 mm
- net Net-(FAN2-Pad2): track 13.0 -> 9.01 mm
- net GND: track 0.00 -> 4.01 mm, vias 0 -> 5
- net /SIGON2: track 9.85 -> 7.12 mm
- net +12V: track 49.1 -> 49.7 mm
- net Net-(FAN1-Pad2): track 13.0 -> 12.5 mm
- net /SIGPWM1: vias 0 -> 1
- added copper zone on B.Cu, net GND
Other:
- board outline added: 25.9 x 42.9 mm
- net class FANPWR added: clearance 0.2, trace_width 0.508, via_dia 0.8, via_drill 0.4
- board text added: "+5V"
- board text added: "3V3"
- board text added: "GND"

Commit message: Change connector for FLOW connector.
Parts:
- FLOW1: footprint Connector_PinHeader_2.54mm:PinHeader_1x02_P2.54mm_Vertical -> Connector_JST:JST_XH_B02B-XH-A_1x02_P2.50mm_Vertical
- moved FLOW1 1.27 mm to (192.4, 87.0), turned to 180 degrees
Routing:
- net /FLOW: track 40.1 -> 41.3 mm
Other:
- board size 25.9 x 42.9 mm -> 25.4 x 44.2 mm
- board text added: "2018-11-27"
- board text added: "Karol Krizka"
Changed lines of the file:
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@@
   (general
     (thickness 1.6)
-    (drawings 8)
+    (drawings 10)
     (tracks 133)
     (zones 0)
@@
       (outputformat 1)
       (mirror false)
-      (drillshape 1)
+      (drillshape 0)
       (scaleselection 1)
-      (outputdirectory ""))
+      (outputdirectory "gerbers/"))
   )
   (net 0 "")
@@
     (add_net "Net-(Q2-Pad3)")
   )
-  (module Connector_PinHeader_2.54mm:PinHeader_1x02_P2.54mm_Vertical (layer F.Cu)
-    (at 193.675 86.995 270)
-    (descr "Through hole straight pin header, 1x02, 2.54mm pitch, single row")
-    (tags "Through hole pin header THT 1x02 2.54mm single row")
-    (fp_text reference FLOW1 (at 2.159 3.683) (layer F.SilkS)
-      (effects (font (size 1 1) (thickness 0.15)))
-    )
-    (fp_text value Conn_01x02 (at 0 4.87 270) (layer F.Fab)
-      (effects (font (size 1 1) (thickness 0.15)))
-    )
-    (fp_line (start -0.635 -1.27) (end 1.27 -1.27) (layer F.Fab) (width 0.1))
-    (fp_line (start 1.27 -1.27) (end 1.27 3.81) (layer F.Fab) (width 0.1))
-    (fp_line (start 1.27 3.81) (end -1.27 3.81) (layer F.Fab) (width 0.1))
-    (fp_line (start -1.27 3.81) (end -1.27 -0.635) (layer F.Fab) (width 0.1))
-    (fp_line (start -1.27 -0.635) (end -0.635 -1.27) (layer F.Fab) (width 0.1))
-    (fp_line (start -1.33 3.87) (end 1.33 3.87) (layer F.SilkS) (width 0.12))
-    (fp_line (start -1.33 1.27) (end -1.33 3.87) (layer F.SilkS) (width 0.12))
-    (fp_line (start 1.33 1.27) (end 1.33 3.87) (layer F.SilkS) (width 0.12))
-    (fp_line (start -1.33 1.27) (end 1.33 1.27) (layer F.SilkS) (width 0.12))
-    (fp_line (start -1.33 0) (end -1.33 -1.33) (layer F.SilkS) (width 0.12))
-    (fp_line (start -1.33 -1.33) (end 0 -1.33) (layer F.SilkS) (width 0.12))
-    (fp_line (start -1.8 -1.8) (end -1.8 4.35) (layer F.CrtYd) (width 0.05))
-    (fp_line (start -1.8 4.35) (end 1.8 4.35) (layer F.CrtYd) (width 0.05))
-    (fp_line (start 1.8 4.35) (end 1.8 -1.8) (layer F.CrtYd) (width 0.05))
-    (fp_line (start 1.8 -1.8) (end -1.8 -1.8) (layer F.CrtYd) (width 0.05))
-    (fp_text user %R (at 0 1.27) (layer F.Fab)
-      (effects (font (size 1 1) (thickness 0.15)))
-    )
-    (pad 1 thru_hole rect (at 0 0 270) (size 1.7 1.7) (drill 1) (layers *.Cu *.Mask)
+  (module Connector_JST:JST_XH_B02B-XH-A_1x02_P2.50mm_Vertical (layer F.Cu)
+    (at 192.405 86.995 180)
+    (descr "JST XH series connector, B02B-XH-A (http://www.jst-mfg.com/product/pdf/eng/eXH.pdf), generated with kicad-footprint-generator")
+    (tags "connector JST XH side entry")
+    (fp_text reference FLOW1 (at -5.08 2.54 180) (layer F.SilkS)
+      (effects (font (size 1 1) (thickness 0.15)))
+    )
+    (fp_text value Conn_01x02 (at 1.25 4.6 180) (layer F.Fab)
+      (effects (font (size 1 1) (thickness 0.15)))
+    )
+    (fp_line (start -2.45 -2.35) (end -2.45 3.4) (layer F.Fab) (width 0.1))
+    (fp_line (start -2.45 3.4) (end 4.95 3.4) (layer F.Fab) (width 0.1))
+    (fp_line (start 4.95 3.4) (end 4.95 -2.35) (layer F.Fab) (width 0.1))
+    (fp_line (start 4.95 -2.35) (end -2.45 -2.35) (layer F.Fab) (width 0.1))
+    (fp_line (start -2.56 -2.46) (end -2.56 3.51) (layer F.SilkS) (width 0.12))
+    (fp_line (start -2.56 3.51) (end 5.06 3.51) (layer F.SilkS) (width 0.12))
+    (fp_line (start 5.06 3.51) (end 5.06 -2.46) (layer F.SilkS) (width 0.12))
+    (fp_line (start 5.06 -2.46) (end -2.56 -2.46) (layer F.SilkS) (width 0.12))
+    (fp_line (start -2.95 -2.85) (end -2.95 3.9) (layer F.CrtYd) (width 0.05))
+    (fp_line (start -2.95 3.9) (end 5.45 3.9) (layer F.CrtYd) (width 0.05))
+    (fp_line (start 5.45 3.9) (end 5.45 -2.85) (layer F.CrtYd) (width 0.05))
+    (fp_line (start 5.45 -2.85) (end -2.95 -2.85) (layer F.CrtYd) (width 0.05))
+    (fp_line (start -0.625 -2.35) (end 0 -1.35) (layer F.Fab) (width 0.1))
+    (fp_line (start 0 -1.35) (end 0.625 -2.35) (layer F.Fab) (width 0.1))
+    (fp_line (start 0.75 -2.45) (end 0.75 -1.7) (layer F.SilkS) (width 0.12))
+    (fp_line (start 0.75 -1.7) (end 1.75 -1.7) (layer F.SilkS) (width 0.12))
+    (fp_line (start 1.75 -1.7) (end 1.75 -2.45) (layer F.SilkS) (width 0.12))
+    (fp_line (start 1.75 -2.45) (end 0.75 -2.45) (layer F.SilkS) (width 0.12))
+    (fp_line (start -2.55 -2.45) (end -2.55 -1.7) (layer F.SilkS) (width 0.12))
+    (fp_line (start -2.55 -1.7) (end -0.75 -1.7) (layer F.SilkS) (width 0.12))
+    (fp_line (start -0.75 -1.7) (end -0.75 -2.45) (layer F.SilkS) (width 0.12))
+    (fp_line (start -0.75 -2.45) (end -2.55 -2.45) (layer F.SilkS) (width 0.12))
+    (fp_line (start 3.25 -2.45) (end 3.25 -1.7) (layer F.SilkS) (width 0.12))
+    (fp_line (start 3.25 -1.7) (end 5.05 -1.7) (layer F.SilkS) (width 0.12))
+    (fp_line (start 5.05 -1.7) (end 5.05 -2.45) (layer F.SilkS) (width 0.12))
+    (fp_line (start 5.05 -2.45) (end 3.25 -2.45) (layer F.SilkS) (width 0.12))
+    (fp_line (start -2.55 -0.2) (end -1.8 -0.2) (layer F.SilkS) (width 0.12))
+    (fp_line (start -1.8 -0.2) (end -1.8 2.75) (layer F.SilkS) (width 0.12))
+    (fp_line (start -1.8 2.75) (end 1.25 2.75) (layer F.SilkS) (width 0.12))
+    (fp_line (start 5.05 -0.2) (end 4.3 -0.2) (layer F.SilkS) (width 0.12))
+    (fp_line (start 4.3 -0.2) (end 4.3 2.75) (layer F.SilkS) (width 0.12))
+    (fp_line (start 4.3 2.75) (end 1.25 2.75) (layer F.SilkS) (width 0.12))
+    (fp_line (start -1.6 -2.75) (end -2.85 -2.75) (layer F.SilkS) (width 0.12))
+    (fp_line (start -2.85 -2.75) (end -2.85 -1.5) (layer F.SilkS) (width 0.12))
+    (fp_text user %R (at 1.25 2.7 180) (layer F.Fab)
+      (effects (font (size 1 1) (thickness 0.15)))
+    )
+    (pad 1 thru_hole rect (at 0 0 180) (size 1.7 2) (drill 1) (layers *.Cu *.Mask)
       (net 24 /FLOW))
-    (pad 2 thru_hole oval (at 0 2.54 270) (size 1.7 1.7) (drill 1) (layers *.Cu *.Mask)
-      (net 17 GND))
-    (model ${KISYS3DMOD}/Connector_PinHeader_2.54mm.3dshapes/PinHeader_1x02_P2.54mm_Vertical.wrl
+    (pad 2 thru_hole oval (at 2.5 0 180) (size 1.7 2) (drill 1) (layers *.Cu *.Mask)
+      (net 17 GND))
+    (model ${KISYS3DMOD}/Connector_JST.3dshapes/JST_XH_B02B-XH-A_1x02_P2.50mm_Vertical.wrl
       (at (xyz 0 0 0))
       (scale (xyz 1 1 1))
@@
     (tags resistor)
     (attr smd)
-    (fp_text reference R6 (at -2.286 0 270) (layer F.SilkS)
+    (fp_text reference R6 (at -1.27 -1.27 270) (layer F.SilkS)
       (effects (font (size 0.508 0.508) (thickness 0.0762)))
     )
@@
     (descr "DC Barrel Jack")
     (tags "Power Jack")
-    (fp_text reference J2 (at -8.128 -5.588 270) (layer F.SilkS)
-      (effects (font (size 1 1) (thickness 0.15)))
+    (fp_text reference J2 (at -8.128 -5.334 270) (layer F.SilkS)
+      (effects (font (size 0.508 0.508) (thickness 0.0762)))
     )
     (fp_text value Conn_01x03 (at -6.2 -5.5 90) (layer F.Fab)
@@
     )
   )
+  (gr_text 2018-11-27 (at 207.137 84.074) (layer F.SilkS)
+    (effects (font (size 1.016 1.016) (thickness 0.127)))
+  )
+  (gr_text "Karol Krizka" (at 195.707 115.062) (layer F.SilkS)
+    (effects (font (size 1.016 1.016) (thickness 0.127)))
+  )
+  (gr_line (start 186.944 83.312) (end 186.944 127.508) (layer Edge.Cuts) (width 0.15))
+  (gr_line (start 212.344 127.508) (end 186.944 127.508) (layer Edge.Cuts) (width 0.15))
+  (gr_line (start 212.344 83.312) (end 212.344 127.508) (layer Edge.Cuts) (width 0.15))
+  (gr_line (start 186.944 83.312) (end 212.344 83.312) (layer Edge.Cuts) (width 0.15))
   (gr_text 3V3 (at 188.214 109.22) (layer F.SilkS)
     (effects (font (size 0.381 0.381) (thickness 0.0762)) (justify right))
@@
     (effects (font (size 0.381 0.381) (thickness 0.0762)) (justify left))
   )
-  (gr_line (start 186.69 127.762) (end 186.69 84.836) (layer Edge.Cuts) (width 0.15))
-  (gr_line (start 212.598 127.762) (end 186.69 127.762) (layer Edge.Cuts) (width 0.15))
-  (gr_line (start 212.598 84.836) (end 212.598 127.762) (layer Edge.Cuts) (width 0.15))
-  (gr_line (start 186.69 84.836) (end 212.598 84.836) (layer Edge.Cuts) (width 0.15))
   (segment (start 208.504 93.98) (end 208.026 93.502) (width 0.25) (layer F.Cu) (net 3))
   (segment (start 209.804 93.98) (end 208.504 93.98) (width 0.25) (layer F.Cu) (net 3))
@@
   (segment (start 196.928 103.124) (end 195.662 104.39) (width 0.508) (layer F.Cu) (net 23))
   (segment (start 197.628 103.124) (end 196.928 103.124) (width 0.508) (layer F.Cu) (net 23))
-  (segment (start 196.5475 86.995) (end 193.675 86.995) (width 0.25) (layer F.Cu) (net 24))
   (segment (start 211.455 106.329) (end 211.104 106.68) (width 0.25) (layer F.Cu) (net 24))
   (segment (start 211.104 106.68) (end 209.804 106.68) (width 0.25) (layer F.Cu) (net 24))
@@
   (segment (start 197.8175 85.725) (end 210.185 85.725) (width 0.25) (layer F.Cu) (net 24))
   (segment (start 196.5475 86.995) (end 197.8175 85.725) (width 0.25) (layer F.Cu) (net 24))
+  (segment (start 192.405 86.995) (end 196.5475 86.995) (width 0.25) (layer F.Cu) (net 24))
   (zone (net 17) (net_name GND) (layer B.Cu) (hatch edge 0.508)
     (connect_pads (clearance 0.508))
@@
     (polygon
       (pts
-        (xy 187.452 85.344) (xy 211.836 85.344) (xy 211.836 127) (xy 187.452 127)
+        (xy 187.452 83.82) (xy 211.836 83.82) (xy 211.836 127) (xy 187.452 127)
       )
     )
